Commit message: Bringup package added

File: ros2_servox_ws/src/servox_description/urdf/servox.xacro (robot description, xacro)
@@ -2,6 +2,12 @@
 <robot name="servox" xmlns:xacro="http://www.ros.org/wiki/xacro">
 <xacro:include filename="$(find servox_description)/urdf/materials.xacro" />
-<xacro:include filename="$(find servox_description)/urdf/servox.ros2control" />
+<xacro:include filename="$(find servox_description)/urdf/servox.ros2_control.xacro" />
 <xacro:include filename="$(find servox_description)/urdf/servox.gazebo" />
+<link name="world"/>
+<joint name="world_to_base" type="fixed">
+  <parent link="world"/>
+  <child link="base_link"/>
+  <origin xyz="0 0 0" rpy="0 0 0"/>
+</joint>
 <link name="base_link">
   <inertial>
