Commit message: hardware_interface added

File: ros2_servox_ws/src/servox_description/urdf/servox.ros2_control.xacro (robot description, xacro)
@@ -1,10 +1,16 @@
 <?xml version="1.0"?>
 <robot xmlns:xacro="http://www.ros.org/wiki/xacro">
-    <xacro:macro name="servox_ros2_control" params="name initial_positions_file">
+    <xacro:macro name="servox_ros2_control" params="name initial_positions_file use_mock:=false">
         <xacro:property name="initial_positions" value="${load_yaml(initial_positions_file)['initial_positions']}"/>
         <ros2_control name="Arm" type="system">
             <hardware>
-                <!-- By default, set up controllers for simulation. This won't work on real hardware -->
-                <plugin>mock_components/GenericSystem</plugin>
+                <xacro:if value="${use_mock}">
+                    <!-- Simulation mode: mock components (no ESP32 needed) -->
+                    <plugin>mock_components/GenericSystem</plugin>
+                </xacro:if>
+                <xacro:unless value="${use_mock}">
+                    <!-- Real hardware mode: communicates with ESP32 via /arm/command & /arm/state -->
+                    <plugin>servox_hardware/ServoXArmHardwareInterface</plugin>
+                </xacro:unless>
             </hardware>
             <joint name="base_joint">

File: ros2_servox_ws/src/servox_moveit_config/config/servox.ros2_control.xacro (robot description, xacro)
@@ -1,10 +1,16 @@
 <?xml version="1.0"?>
 <robot xmlns:xacro="http://www.ros.org/wiki/xacro">
-    <xacro:macro name="servox_ros2_control" params="name initial_positions_file">
+    <xacro:macro name="servox_ros2_control" params="name initial_positions_file use_mock:=false">
         <xacro:property name="initial_positions" value="${load_yaml(initial_positions_file)['initial_positions']}"/>
         <ros2_control name="${name}" type="system">
             <hardware>
-                <!-- By default, set up controllers for simulation. This won't work on real hardware -->
-                <plugin>mock_components/GenericSystem</plugin>
+                <xacro:if value="${use_mock}">
+                    <!-- Simulation mode: mock components (no ESP32 needed) -->
+                    <plugin>mock_components/GenericSystem</plugin>
+                </xacro:if>
+                <xacro:unless value="${use_mock}">
+                    <!-- Real hardware mode: communicates with ESP32 via /arm/command & /arm/state -->
+                    <plugin>servox_hardware/ServoXArmHardwareInterface</plugin>
+                </xacro:unless>
             </hardware>
             <joint name="base_joint">
